File: PCB/UVCleanPCB-backups/UVCleanPCB-2025-02-18_022517/UVCleanPCB.kicad_sch (KiCad schematic)
At the start: 61 parts, among them IC1 L78L33ACUTR, J1 Conn_01x04_Pin, J2 Conn_01x02_Pin, J3 Conn_01x02_Pin, Q1 IRLML2402, Q2 IRLML2402, SW1 SW_SPDT, SW3 SW_Push, SW4 SW_Push, SW5 SW_Push_SPDT, U1 STM32L031K6Tx, U10 LM7806_TO220, U2 LSM6DS3, U3 74HC74D_652, U4 MCP73831-2-MC, U6 KL265-50W-SM-WD, U7 KL265-50W-SM-WD

Commit message: PCB layout
Parts:
- removed C16: 330n, Capacitor_SMD:C_0603_1608Metric, symbol Device:C
- removed C17: 100n, Capacitor_SMD:C_0603_1608Metric, symbol Device:C
- removed D8: LED, LED_SMD:LED_0603_1608Metric, symbol Device:LED
- removed IC1: L78L33ACUTR, UVCLibrary:LDK320ADU30R, symbol UVCLED:L78L33ACUTR
- removed Q1, Q2: IRLML2402, UVCLibrary:SOT-23, symbol UVCLED:IRLML2402
- removed R6: 100R, Resistor_SMD:R_0402_1005Metric, symbol Device:R
- removed R7: 600k, Resistor_SMD:R_0603_1608Metric, symbol Device:R
- removed SW4: SW_Push, Button_Switch_SMD:SW_Tactile_SPST_NO_Straight_CK_PTS636Sx25SMTRLFS, symbol Switch:SW_Push
- removed SW5: SW_Push_SPDT, Button_Switch_SMD:SW_SPDT_CK_JS102011SAQN, symbol Switch:SW_Push_SPDT
- removed U10: LM7806_TO220, Package_TO_SOT_THT:TO-220-3_Vertical, symbol Regulator_Linear:LM7806_TO220
- removed U3: 74HC74D_652, UVCLibrary:SOIC127P600X175-14N, symbol UVCLED:74HC74D_652
- removed U6, U7: KL265-50W-SM-WD, UVCLibrary:3535, symbol UVCLED:KL265-50W-SM-WD
- added C13: 0.1u, Capacitor_SMD:C_0603_1608Metric, symbol Device:C
- added C15: 22u, Capacitor_SMD:C_1206_3216Metric, symbol Device:C
- added D1, D3: LED, symbol Device:LED
- added L1: 4.7u, Inductor_SMD:L_Vishay_IHLP-2525, symbol Device:L
- added Q1, Q2: IRLML0030, Package_TO_SOT_SMD:SOT-23, symbol Transistor_FET:IRLML0030
- added R3, R4: 100k, Resistor_SMD:R_0603_1608Metric, symbol Device:R
- added SW2: SW_Push, symbol Switch:SW_Push
- added U3: AP63203WU, Package_TO_SOT_SMD:TSOT-23-6, symbol Regulator_Switching:AP63203WU
- C10, C11, C19, C20, C21: footprint Capacitor_SMD:C_0402_1005Metric -> (none)
- C12: value 0.33u -> 22u
- C14: value 0.1u -> 22u
- C18: value 5u -> 100n; footprint Capacitor_SMD:C_0805_2012Metric -> (none)
- D4, D5: footprint LED_SMD:LED_0603_1608Metric -> (none)
- D6: footprint LED_SMD:LED_0402_1005Metric -> (none)
- R11, R2, R5: footprint Resistor_SMD:R_0402_1005Metric -> (none)
- R15, R16: value 100R -> 1k; footprint Resistor_SMD:R_0402_1005Metric -> (none)
- R17: value 1M -> 10k; footprint Resistor_SMD:R_0603_1608Metric -> (none)
- SW1: footprint Button_Switch_SMD:SW_SPDT_PCM12 -> Button_Switch_THT:SW_E-Switch_EG1224_SPDT_Angled
- SW3: footprint Button_Switch_SMD:SW_Tactile_SPST_NO_Straight_CK_PTS636Sx25SMTRLFS -> (none)
- U4: footprint Package_TO_SOT_SMD:SOT-23-8 -> Package_TO_SOT_SMD:SOT-23-5
Connections:
- net +6V is gone; now on net B+: R14.1, R9.1
- net B+ PWRBTN is gone; now on net B+: C12.1
- net +3.3V: now also C1.1, C14.1, C18.1, C19.1, C2.1, C20.2, C21.1, C3.1, C4.1, C5.1, C8.1, FB1.2, J1.1 (Pin_1), R15.1, R18.2, R19.2, R20.2, SW3.1, U1.1 (VDD), U1.10 (PA4), U1.17 (VDD), U1.8 (PA2), U2.5 (VDDIO), U2.8 (VDD), C15.1, L1.2, SW2.1, U3.1 (FB)
- net B+: now also D2.2 (A), J2.1 (Pin_1), R3.1, R3.2, R4.1, U3.2 (EN), U3.3 (IN)
- net GND: now also R11.2, C15.2, Q1.3 (D), Q2.3 (D), R4.2, U3.4 (GND)
- net at R17.1, SW3.2: no longer C18.1
- net at R10.2, R8.1: now also Q1.1 (G)
- net at R14.2: now also D3.2 (A)
- net at R9.2: now also D1.2 (A)
- net at R12.2, R13.1: now also Q2.1 (G)
- removed net +3V3: C1.1, C14.1, C2.1, C20.2, C21.1, C3.1, C4.1, C5.1, J1.1 (Pin_1), R11.1, R15.1, R18.2, R19.2, R20.2, U1.1 (VDD), U1.17 (VDD), U2.5 (VDDIO), U2.8 (VDD)
- net +3V3A renamed +3.3VA
- net +3.3VA: no longer C8.1, FB1.2
- removed net A4_USER_BTN: C19.1, R11.2, U1.10 (PA4)
- net A7_STATUS_LED2: no longer names the net of U1.13 (PA7)
- new net: C13.1, U3.6 (BST)
- new net: C13.2, L1.1, U3.5 (SW)
- new net: D3.1 (K), Q2.2 (S)
- new net: R11.1, SW2.2
- new net: D1.1 (K), Q1.2 (S)
- no-connect marks 22 -> 13
Other:
- note added: "UVClean PCB"
- note removed: "6V REGULATOR"
- note removed: "STATUS LED 2"
- note removed: "UVC disinfection PCB"
- title: UVC disinfection PCB -> UVClean PCB
- moved on the sheet: C1, C10, C11, C12, C14, C2, C20, C21, C3, C4, C5, C6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
